File: board/wall-e.kicad_pcb (KiCad board)
At the start: 2 copper layers, 78.7 x 64.4 mm, 63 parts, among them J1 Raspberry_Pi_2_3, J10 PCA9685, J11 VL53L0X, J12 VL53L0X, J13 VL53L0X, J14 MotorDrv2, J15 Motor2, J16 IMU, J17 INA219, J18 INA219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

Commit message: Tweaks
Parts:
- added J19: GS2, Connectors:GS2, B.Cu at (65.6, 33.2)
- moved C12 3.32 mm to (78.7, 36.0), turned to 180 degrees
- moved C11 1.36 mm to (74.7, 58.6)
- moved R1 0.89 mm to (89.2, 52.2)
- moved C9 0.86 mm to (74.7, 71.2)
- moved C4 0.46 mm to (91.4, 58.2)
Routing:
- net +5V: track 70.6 -> 80.3 mm
- net GNDA: track 11.8 -> 21.2 mm, vias 4 -> 5
- net +3V3: track 179.4 -> 172.7 mm, vias 11 -> 13
- net GND: track 25.4 -> 28.4 mm, vias 11 -> 13
- net I2C_M6_SCLK: track 12.6 -> 14.6 mm
- net PI_RX: track 53.1 -> 52.0 mm
- net I2C_M7_SDA: track 43.8 -> 42.7 mm
- net PI_I2C_SDA: track 25.0 -> 26.0 mm
- net PI_I2C_SCLK: track 21.8 -> 22.8 mm
- net PROP_RES: track 2.90 -> 3.67 mm
- net I2C_M7_SCLK: track 41.8 -> 41.1 mm
- net I2C_ISO_SDA: track 35.6 -> 35.0 mm
Other:
- net class Default: clearance 0.25 -> 0.2
- rule trace_clearance: 0.25 -> 0.2
